File: Kicad/Envirotector.kicad_pcb (KiCad board)
At the start: 2 copper layers, 3 parts, among them J1 OLED Display, U1 XIAO-RP2040-DIP, U2 DHT11

Commit message: Upload
Parts:
- added G***: LOGO, LOGO, B.Cu at (90.3, 121.3)
- added G***: LOGO, LOGO, B.Cu at (133.3, 72.8)
- added G***: LOGO, LOGO, B.Cu at (106.6, 91.1)
- added G***: LOGO, LOGO, B.Cu at (133.0, 118.0)
- added J2: Micro_SD_Card, Connector_Card:microSD_HC_Hirose_DM3AT-SF-PEJM5, F.Cu at (130.9, 66.6)
- added SW1: RotaryEncoder_Switch, Rotary_Encoder:RotaryEncoder_Alps_EC11E-Switch_Vertical_H20mm, F.Cu at (123.2, 120.2)
- added U3: ~, LARGE:RTC_DS3231, F.Cu at (72.7, 113.7)
- added U4: ~, SPARK:BMP180, F.Cu at (81.2, 124.5)
- moved U2 75.4 mm to (103.6, 118.2)
- moved U1 67.1 mm to (109.6, 68.2)
- moved J1 38.3 mm to (126.6, 97.8), turned to 90 degrees
Connections:
- U1 pad 1: Net-(U1-GPIO26/ADC0/A0) -> Net-(J2-DAT3/CD)
- U1 pad 10: unconnected-(U1-GPIO4/MISO-Pad10) -> Net-(J2-DAT0)
- U1 pad 11: unconnected-(U1-GPIO3/MOSI-Pad11) -> Net-(J2-CMD)
- U1 pad 2: unconnected-(U1-GPIO27/ADC1/A1-Pad2) -> Net-(U1-GPIO27/ADC1/A1)
- U1 pad 3: unconnected-(U1-GPIO28/ADC2/A2-Pad3) -> Net-(U1-GPIO28/ADC2/A2)
- U1 pad 4: unconnected-(U1-GPIO29/ADC3/A3-Pad4) -> Net-(U1-GPIO29/ADC3/A3)
- U1 pad 7: unconnected-(U1-GPIO0/TX-Pad7) -> Net-(U1-GPIO0/TX)
- U1 pad 9: unconnected-(U1-GPIO2/SCK-Pad9) -> Net-(J2-CLK)
- U2 pad 2: Net-(U1-GPIO26/ADC0/A0) -> Net-(U1-GPIO0/TX)
Routing:
- net GND: track 0.00 -> 240.6 mm, vias 0 -> 1
- net Net-(J1-Pin_1): track 0.00 -> 189.6 mm, vias 0 -> 2
- net Net-(J1-Pin_2): track 0.00 -> 117.8 mm, vias 0 -> 1
- net +5V: track 0.00 -> 99.9 mm
- net +3.3V: track 0.00 -> 86.1 mm, vias 0 -> 2
- net Net-(U1-GPIO29/ADC3/A3): track 0.00 -> 77.7 mm
- net Net-(U1-GPIO27/ADC1/A1): track 0.00 -> 72.7 mm
- net Net-(U1-GPIO28/ADC2/A2): track 0.00 -> 66.0 mm
- net Net-(U1-GPIO0/TX): track 0.00 -> 49.5 mm, vias 0 -> 1
- net Net-(J2-DAT3/CD): track 0.00 -> 37.6 mm, vias 0 -> 2
- net Net-(J2-DAT0): track 0.00 -> 25.7 mm
- net Net-(J2-CLK): track 0.00 -> 18.9 mm, vias 0 -> 2
- net Net-(J2-CMD): track 0.00 -> 15.9 mm
Other:
- board outline added: 75 x 77.7 mm
- board text added: "ENVIROTECTOR V1"
